Commit message: Second commit

File: ros2_ws/install/quadruped_mujoco/share/quadruped_mujoco/urdf/yobotics.urdf (robot description, URDF)
Before this commit: robot yobotics_description, 25 links, 24 joints
Links:
- removed link FL_calf
- removed link FL_foot
- removed link FL_hip
- removed link FL_thigh
- removed link FR_calf
- removed link FR_foot
- removed link FR_hip
- removed link FR_thigh
- removed link RL_calf
- removed link RL_foot
- removed link RL_hip
- removed link RL_thigh
- removed link RR_calf
- removed link RR_foot
- removed link RR_hip
- removed link RR_thigh
- removed link camera_depth_frame
- removed link camera_depth_optical_frame
- removed link camera_link
- removed link camera_rgb_frame
- removed link camera_rgb_optical_frame
- removed link hokuyo_frame
- removed link imu_link
- removed link trunk
- removed link trunk_interia
Joints:
- removed joint FL_calf_joint
- removed joint FL_foot_fixed
- removed joint FL_hip_joint
- removed joint FL_thigh_joint
- removed joint FR_calf_joint
- removed joint FR_foot_fixed
- removed joint FR_hip_joint
- removed joint FR_thigh_joint
- removed joint RL_calf_joint
- removed joint RL_foot_fixed
- removed joint RL_hip_joint
- removed joint RL_thigh_joint
- removed joint RR_calf_joint
- removed joint RR_foot_fixed
- removed joint RR_hip_joint
- removed joint RR_thigh_joint
- removed joint camera_depth_joint
- removed joint camera_depth_optical_joint
- removed joint camera_joint
- removed joint camera_rgb_joint
- removed joint camera_rgb_optical_joint
- removed joint hokuyo_joint
- removed joint imu_joint
- removed joint trunk_to_trunk_inertia
